File: hardware/RasperryPirateButtons.sch (KiCad schematic (older format))
At the start: 18 parts, among them P1 CONN_01X04, P11 CONN_20X2, P2 CONN_01X04, P3 CONN_01X04, P4 CONN_01X04, Q1 MMBT3904, Q2 MMBT3904, Q3 MMBT3904, Q4 MMBT3904

Commit message: Version 2 of pirate buttons
Parts:
- removed Q1, Q2, Q3, Q4: MMBT3904, TO_SOT_Packages_SMD:SOT-23_Handsoldering, symbol MMBT3904
- added L-B3: LED-B, LEDs:LED-0805, symbol LED
- added L-G4: LED-G, LEDs:LED-0805, symbol LED
- added L-R1: LED-R, LEDs:LED-0805, symbol LED
- added L-W2: LED-W, LEDs:LED-0805, symbol LED
- added Q1, Q2, Q3, Q4: AO3400, TO_SOT_Packages_SMD:SOT-23, symbol BSS138
- added R11, R12, R13, R14: 560, Resistors_SMD:R_0805_HandSoldering, symbol R
- added SW1, SW2, SW3, SW4: BG SW, lib:AB2_PB_MOM_6MM_PTH_BLK, symbol SW_PUSH_SMALL
- R1, R2, R3, R4: value 470 -> 100K; footprint Resistors_SMD:R_0603_HandSoldering -> Resistors_SMD:R_0805_HandSoldering
Connections:
- net +12V: now also R11.2, R12.2, R13.2, R14.2
- net GND: now also R1.2, R2.2, R3.2, R4.2, Q1.2 (S), Q2.2 (S), Q3.2 (S), Q4.2 (S), SW1.2, SW2.2, SW3.2, SW4.2
- net GPIO05: now also Q3.1 (G)
- net GPIO06: now also SW3.1
- net GPIO13: now also Q4.1 (G)
- net GPIO17: now also Q1.1 (G)
- net GPIO23: now also Q2.1 (G)
- net GPIO24: now also SW2.1
- net GPIO26: now also SW4.1
- net GPIO27: now also SW1.1
- net at P1.2 (P2): now also L-R1.1 (K), Q1.3 (D)
- net at P2.2 (P2): now also L-W2.1 (K), Q2.3 (D)
- net at P3.2 (P2): now also L-B3.1 (K), Q3.3 (D)
- net at P4.2 (P2): now also L-G4.1 (K), Q4.3 (D)
- new net: L-R1.2 (A), R11.1
- new net: L-B3.2 (A), R13.1
- new net: L-W2.2 (A), R12.1
- new net: L-G4.2 (A), R14.1
- no-connect marks 24 -> 28
